Commit message: init tri roller env

File: assets/triroller/objects/urdf/cube_multicolor_rrc.urdf (robot description, URDF)
Before this commit: robot object, 1 links, 0 joints
Links:
- link object: geometry collision box size=0.04 0.04 0.04; visual mesh filename=meshes/cube_multicolor.obj scale=.04 .04 .04

File: assets/triroller/robot_properties_fingers/urdf/high_table_boundary.urdf (robot description, URDF)
Before this commit: robot stage, 1 links, 0 joints
Links:
- link stage_link: geometry collision mesh filename=package://robot_properties_fingers/meshes/high_table_bounda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 scale=0.6 0.6 0.6; visual mesh filename=package://robot_properties_fingers/meshes/high_table_bounda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 scale=0.6 0.6 0.6
