Commit message: change env params, add fly away check

File: assets/biroller/robot_properties_fingers/urdf/biroller.urdf (robot description, URDF)
Before this commit: robot , 17 links, 16 joints
Links:
- added link base, mass 0.0
- link l3: geometry collision mesh filename=package://robot_properties_fingers/meshes/roller_rough.obj scale=1 1 1; visual mesh filename=package://robot_properties_fingers/meshes/roller_rough.obj scale=1 1 1
- link r3: geometry collision mesh filename=package://robot_properties_fingers/meshes/roller_rough.obj scale=1 1 1; visual mesh filename=package://robot_properties_fingers/meshes/roller_rough.obj scale=1 1 1
Joints:
- added joint wrist: type revolute, parent base, child forearm, origin xyz=0.00000 0.00000 0.00 rpy=0.00000 -0.00000 0.00000, axis 0.00000 0.00000 1.00000

Commit message: change to rough gripper

File: assets/biroller/robot_properties_fingers/urdf/biroller.urdf (robot description, URDF)
Before this commit: robot , 17 links, 16 joints
Links:
- link l3: geometry collision mesh filename=package://robot_properties_fingers/meshes/roller_rough.obj scale=1 1 1; visual mesh filename=package://robot_properties_fingers/meshes/roller_rough.obj scale=1 1 1
- link r3: geometry collision mesh filename=package://robot_properties_fingers/meshes/roller_rough.obj scale=1 1 1; visual mesh filename=package://robot_properties_fingers/meshes/roller_rough.obj scale=1 1 1
