Commit message: physical params for constrained control works now

File: assets/biroller/objects/urdf/rounded_cube.urdf (robot description, URDF)
Before this commit: robot object, 1 links, 0 joints
Links:
- link object: geometry collision mesh filename=meshes/rounded_cube.stl scale=0.9 0.9 0.9; visual mesh filename=meshes/rounded_cube.stl scale=0.9 0.9 0.9

File: assets/biroller/robot_properties_fingers/urdf/biroller.urdf (robot description, URDF)
Before this commit: robot , 17 links, 16 joints
Links:
- link l3: mass 0.1 -> 0.01
- link r3: mass 0.1 -> 0.01

Commit message: update parameters

File: assets/biroller/objects/urdf/rounded_cube.urdf (robot description, URDF)
Before this commit: robot object, 1 links, 0 joints
Links:
- link object: geometry collision mesh filename=meshes/rounded_cube.stl scale=1.20 1.20 1.20; visual mesh filename=meshes/rounded_cube.stl scale=1.20 1.20 1.20

File: assets/biroller/robot_properties_fingers/urdf/biroller_wrist.urdf (robot description, URDF)
Before this commit: robot , 17 links, 16 joints
Links:
- added link base, mass 0.0
- link l3: mass 0.01 -> 0.1; geometry collision cylinder length=0.05 radius=0.025; visual cylinder length=0.05 radius=0.025
- link r3: mass 0.01 -> 0.1; geometry collision cylinder length=0.05 radius=0.025; visual cylinder length=0.05 radius=0.025
Joints:
- added joint wrist: type revolute, parent base, child forearm, origin xyz=0.00000 0.00000 0.00000 rpy=0.00000 -0.00000 0.00000, axis 0.00000 0.00000 1.00000, limit lower=-1000 upper=1000 effort=1000.0 velocity=100
- joint roll_l: origin xyz=0.00000 0.01840 0.00000 rpy=0.00000 -0.00000 0.00000 -> xyz=0.00000 0.01840 0.00000 rpy=0.00000 1.57000 0.00000
- joint roll_r: origin xyz=0.00000 -0.01840 0.00000 rpy=0.00000 -0.00000 0.00000 -> xyz=0.00000 -0.01840 0.00000 rpy=0.00000 1.57000 0.00000
